File: pcb/fluke-ir-cable.kicad_sch (KiCad schematic)
At the start: 19 parts, among them J1 USB_C_Receptacle_USB2.0_16P, Q1 SFH3201, U1 LM393, U2 FT232BM

Commit message: Layout
Parts:
- removed Q1: SFH3201, OptoDevice:Osram_SFH9x0x, symbol Sensor_Optical:SFH3201
- added C4: 0.1u, Capacitor_SMD:C_0603_1608Metric_Pad1.08x0.95mm_HandSolder, symbol Device:C
- added Q2: INL-5ANPT30, LED_THT:LED_D5.0mm_Clear, symbol Sensor_Optical:BPW40
- D1: value IR204A -> TSAL6400; footprint LED_THT:LED_D3.0mm_IRBlack -> LED_THT:LED_D5.0mm_Clear
- J1: footprint (none) -> Connector_USB:USB_C_Receptacle_GCT_USB4105-xx-A_16P_TopMnt_Horizontal
- U1: footprint (none) -> Package_SO:TSSOP-8_4.4x3mm_P0.65mm
Connections:
- net GND: now also C4.2, Q2.2 (E)
- net VBUS: now also C4.1
- net at R9.2, U1.5 (+): now also Q2.1 (C)
